File: Voyager60.sch (KiCad schematic (older format))
At the start: 261 parts, among them Q1 2N7002, SW1 5.2x5.2mm, U1 ATmega32U4-MU, U2 PRTR5V0U2X, Y1 16Mhz

Commit message: bete
Parts:
- removed C1, C10, C11, C12, C13, C14, C15, C16, C17, C18, C19, C20, C21, C9: 0.1uF, Capacitors_SMD:C_0603, symbol Device:C_Small
- removed D1, D10, D11, D12, D13, D14, D16, D17, D18, D19, D2, D20, D21, D22, D23, D24, D25, D26, D27, D28, D29, D3, D30, D31, D32, D33, D34, D35, D36, D37, D38, D39, D4, D40, D41, D42, D43, D44, D45, D46, D47, D48, D49, D5, D50, D51, D52, D53, D54, D55, D56, D57, D58, D59, D6, D60, D61, D62, D63, D64, D65, D67, D68, D7, D8, D9: SOD-123, Diodes_SMD:D_SOD-123, symbol Device:D_Small
- removed K_#1, K_#10, K_#2, K_#3, K_#4, K_#5, K_#6, K_#7, K_#8, K_#9, K_'1, K_,1, K_-1, K_.1, K_/1, K_;1, K_=1, K_A1, K_B1, K_C1, K_D1, K_E1, K_ESC1, K_F1, K_G1, K_H1, K_I1, K_J1, K_K1, K_L1, K_M1, K_N1, K_O1, K_P1, K_Q1, K_R1, K_RWIN3, K_S1, K_SBACK1, K_SBACK2, K_SHIFT3, K_SRSHIFT2, K_T1, K_U1, K_V1, K_W1, K_X1, K_Y1, K_Z1, K_[1, K_\2, K_]1: MX-1U, MX_Alps_Hybrid:MX-1U, symbol MX_Alps_Hybrids:MX-1U
- removed K_ALT1, K_CTRL1, K_RCTRL2, K_RWIN2, K_SHIFT2, K_WIN1: MX-1.25U, MX_Alps_Hybrid:MX-1.25U, symbol MX_Alps_Hybrids:MX-1U
- removed K_ALT2, K_CTRL2, K_RALT3, K_RCTRL3: MX-1.5U, MX_Alps_Hybrid:MX-1.5U-FLIPPED, symbol MX_Alps_Hybrids:MX-1U
- removed K_BACK1: MX-2U, MX_Alps_Hybrid:MX-2U, symbol MX_Alps_Hybrids:MX-1U
- removed K_CAPS1, K_SRSHIFT1: MX-1.75U, MX_Alps_Hybrid:MX-1.75U, symbol MX_Alps_Hybrids:MX-1U
- removed K_CAPS2, K_RALT2, K_RMENU2, K_SPACE5: MX-1.25U, MX_Alps_Hybrid:MX-1.25U-FLIPPED, symbol MX_Alps_Hybrids:MX-1U
- removed K_ENTER1, K_SHIFT1: MX-2.25U, MX_Alps_Hybrid:MX-2.25U, symbol MX_Alps_Hybrids:MX-1U
- removed K_ENTER2: MX-ISO, MX_Alps_Hybrid:MX-ISO-ReversedStabilizers, symbol MX_Alps_Hybrids:MX-1U
- removed K_RSHIFT1: MX-2.75U, MX_Alps_Hybrid:MX-2.75U-FLIPPED, symbol MX_Alps_Hybrids:MX-1U
- removed K_SPACE1: MX-7U, MX_Alps_Hybrid:MX-7U-ReversedStabilizers, symbol MX_Alps_Hybrids:MX-1U
- removed K_SPACE2: MX-6.25U, MX_Alps_Hybrid:MX-6.25U-ReversedStabilizers, symbol MX_Alps_Hybrids:MX-1U
- removed K_SPACE3: MX-2.25U, MX_Alps_Hybrid:MX-2.25U-ReversedStabilizers, symbol MX_Alps_Hybrids:MX-1U
- removed K_SPACE4: MX-2.75U, MX_Alps_Hybrid:MX-2.75U-ReversedStabilizers, symbol MX_Alps_Hybrids:MX-1U
- removed K_TAB1, K_\1: MX-1.5U, MX_Alps_Hybrid:MX-1.5U, symbol MX_Alps_Hybrids:MX-1U
- removed K_WIN2: MX-1U, MX_Alps_Hybrid:MX-1U-FLIPPED, symbol MX_Alps_Hybrids:MX-1U
- removed Q1: 2N7002, TO_SOT_Packages_SMD:SOT-23, symbol Transistor_FET:2N7002
- removed R1, R10, R11, R12, R13, R14, R16, R17, R18, R19, R2, R20, R21, R22, R23, R24, R25, R26, R27, R28, R29, R3, R30, R31, R32, R33, R34, R35, R36, R37, R38, R39, R4, R40, R41, R42, R43, R44, R45, R46, R47, R48, R49, R5, R50, R51, R52, R53, R54, R55, R56, R57, R58, R59, R6, R60, R61, R62, R63, R64, R65, R69, R7, R72, R75, R8, R9: 1k, Resistors_SMD:R_0805, symbol Device:R_Small
- removed RGB1, RGB10, RGB11, RGB12, RGB13, RGB14, RGB2, RGB3, RGB4, RGB5, RGB6, RGB7, RGB8, RGB9: WS2812B, WS2812B:WS2812B, symbol ws2812b:WS2812B
- added C?: 0.47uF, Capacitors_SMD:C_0603, symbol Device:C_Small
- added D? (x9): LED_ARGB, symbol Device:LED_ARGB
- added IC?: IS31FL3733-TQLS4, QFP50P900X900X120-49N, symbol SamacSys_Parts:IS31FL3733-TQLS4
- added IC?: ATMEGA32U4-AU, QFP80P1200X1200X120-44N, symbol SamacSys_Parts:ATMEGA32U4-AU
- added J? (x2): AudioJack4, symbol Connector:AudioJack4
- added R?: 20k, Resistors_SMD:R_0805, symbol Device:R_Small
- added R? (x2): 100k, Resistors_SMD:R_0805, symbol Device:R_Small
- added R? (x2): 1k, Resistors_SMD:R_0805, symbol Device:R_Small
- added SW? (x9): SW_Push, symbol Switch:SW_Push
- USB1: symbol Type-C:HRO-TYPE-C-31-M-12 -> Voyager60-rescue:HRO-TYPE-C-31-M-12-Type-C
Connections:
- net labels added: AUDIO, LEDCOL1, LEDCOL2, LEDCOL3, LEDROW1, LEDROW10, LEDROW11, LEDROW12, LEDROW2, LEDROW3, LEDROW4, LEDROW5, LEDROW6, LEDROW7, LEDROW8, LEDROW9, RE1A, RE1B, RE1S, RE2A, RE2B, RE2S, RE3A, RE3B, RE3S, SCL, SDA, SERIAL, SSL
- net labels removed: COL0, COL10, COL11, COL12, COL13, COL4, COL5, COL6, COL7, COL8, COL9, LEDGND, RGBLED, ROW0, ROW4
- wire segments 788 -> 135
- no-connect marks 2 -> 46
Other:
- note added: "TX0(LED)"
- moved on the sheet: C2, C3, C4, C5, C6, C7, C8, F1, R67, R68, R70, R71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
